File: pcbs/left_main_routed.kicad_pcb (KiCad board)
At the start: 2 copper layers, 105.8 x 90.5 mm, 49 parts, among them J2 TRRS, J4 I2C Breakout, J9 Male 9pin, SW18 Val**, SW19 Val**, SW20 Val**, SW21 Val**, SW22 Val**, SW23 Val**, SW24 Val**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

Commit message: V2
Parts:
- added H14: M2, kbd:M2_HOLE_v3, F.Cu at (-44.0, -4.50)
- added H16: M2, kbd:M2_HOLE_v3, F.Cu at (-57.0, 3.50)
- added J10: SCL, kbd:Jumper, F.Cu at (-28.0, -50.0)
- added J15: Male 9pin, Library:kb_90deg_connector_male_9pin, F.Cu at (-6.30, 16.1)
- added J8: SERIAL, kbd:Jumper, F.Cu at (-28.0, -54.0)
- J9: value Male 9pin -> SDA; footprint Library:kb_90deg_connector_male_9pin -> kbd:Jumper
- moved J9 71.1 mm to (-28.0, -52.0), turned to 180 degrees
Connections:
- J2 pad 2: GND -> VCC
- J2 pad 3: SERIAL -> TRRS3
- J2 pad 4: VCC -> TRRS4
- J9 pad 1: VCC -> SDA
- J9 pad 2: GND -> TRRS4
Routing:
- net R5: track 105.4 -> 226.5 mm, vias 2 -> 1
- net R4: track 104.2 -> 223.7 mm
- net scroll_r2: track 107.3 -> 221.6 mm, vias 2 -> 1
- net scroll_switch: track 108.2 -> 216.2 mm, vias 2 -> 0
- net scroll_r1: track 109.7 -> 211.6 mm, vias 2 -> 1
- net R3: track 226.3 -> 140.4 mm, vias 3 -> 1
- net SERIAL: track 67.8 -> 23.2 mm
- net TRRS3: track 0.00 -> 43.2 mm
- net C5: track 100.2 -> 140.3 mm, vias 2 -> 0
- net TRRS4: track 0.00 -> 38.1 mm, vias 0 -> 2
- net R1: track 132.9 -> 107.3 mm
- net GND: track 42.4 -> 18.0 mm, vias 3 -> 6
- net rgb_ug5_out: track 45.9 -> 34.9 mm, vias 0 -> 2
- net C3: track 58.4 -> 48.0 mm, vias 1 -> 0
- net SDA: track 82.7 -> 92.1 mm, vias 0 -> 1
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Other:
- board size 105.8 x 90.5 mm -> 106.2 x 90.5 mm
- board text added: "GND"
- board text added: "SCL"
- board text added: "SDA"
- board text added: "VCC"
