File: pcbs/right_main_routed.kicad_pcb (KiCad board)
At the start: 2 copper layers, 105.8 x 90.5 mm, 49 parts, among them J1 TRRS, J3 I2C Breakout, J8 Male 9pin, SW1 Val**, SW10 Val**, SW11 Val**, SW12 Val**, SW13 Val**, SW14 Val**, SW15 Val**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

Commit message: V2
Parts:
- removed J8: Male 9pin, Library:kb_90deg_connector_male_9pin
- added H13: M2, kbd:M2_HOLE_v3, F.Cu at (49.0, -4.50)
- added H15: M2, kbd:M2_HOLE_v3, F.Cu at (62.0, 3.50)
- added J14: Male 9pin, Library:kb_90deg_connector_male_9pin, F.Cu at (11.3, 16.1)
- added J5: SERIAL, kbd:Jumper, F.Cu at (33.0, -54.0)
- added J6: SDA, kbd:Jumper, F.Cu at (33.0, -52.0)
- added J7: SCL, kbd:Jumper, F.Cu at (33.0, -50.0)
Connections:
- J1 pad 2: GND -> VCC
- J1 pad 3: SERIAL -> TRRS3
- J1 pad 4: VCC -> TRRS4
Routing:
- net R2: track 178.8 -> 120.7 mm
- net TRRS3: track 0.00 -> 44.1 mm
- net GND: track 19.6 -> 62.3 mm, vias 2 -> 0
- net TRRS4: track 0.00 -> 41.2 mm, vias 0 -> 2
- net SERIAL: track 58.9 -> 18.3 mm
- net R3: track 185.7 -> 145.9 mm, vias 0 -> 1
- net scroll_r2: track 85.7 -> 103.1 mm, vias 1 -> 0
- net VCC: track 30.9 -> 13.9 mm
- net SDA: track 89.0 -> 97.0 mm
- net scroll_r1: track 91.0 -> 99.0 mm, vias 1 -> 2
- net C2: track 116.6 -> 109.4 mm
- net R1: track 129.6 -> 135.8 mm, vias 0 -> 1
- net scroll_switch: track 89.1 -> 94.9 mm, vias 2 -> 0
- net SCL: track 93.0 -> 98.5 mm
- net rgb_ug2_out: track 36.7 -> 31.5 mm
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Other:
- board size 105.8 x 90.5 mm -> 106.2 x 90.5 mm
- board text added: "GND"
- board text added: "SCL"
- board text added: "SDA"
- board text added: "VCC"
